Commit message: Imported upstream version '0.6.4' of 'upstream'

File: cob_hardware_config/raw3-3/urdf/raw3-3.urdf.xacro (robot description, xacro)
@@ -35,3 +35,20 @@
   </xacro:lookat>
 -->
+  <!-- scan top mount -->
+    <joint name="base_laser_top_joint" type="fixed" >
+      <origin xyz="0.28 0.0 0.885" rpy="0.0 0.0 ${M_PI}" />
+      <parent link="base_link" />
+      <child link="base_laser_top_link" />
+    </joint>
+    <link name="base_laser_top_link">
+    <xacro:default_inertial />
+    <visual>
+      <origin xyz="0.0 0.0 0.0" rpy="0.0 0.0 0.0" />
+      <geometry>
+      <box size="0.10 0.03 0.03" />
+      </geometry>
+      <material name="IPA/Black" />
+    </visual>
+    </link>
+  <!-- END: scan top mount -->
 </robot>
