Commit message: Imported upstream version '0.6.5' of 'upstream'

File: cob_hardware_config/cob3-9/urdf/calibration_default.urdf.xacro (robot description, xacro)
@@ -50,10 +50,10 @@
 	<property name="def_head_yaw" value="0.0"/>
 	<!-- arm mount positions | relative to base_link -->
-	<property name="def_arm_x" value="0.040"/>
+	<property name="def_arm_x" value="-0.004"/>
 	<property name="def_arm_y" value="-0.065"/>
-	<property name="def_arm_z" value="0.85"/>
-	<property name="def_arm_roll" value="-0.1"/>
-	<property name="def_arm_pitch" value="-3.896992654"/>
-	<property name="def_arm_yaw" value="1.33899265359"/>
+	<property name="def_arm_z" value="0.83357"/>
+	<property name="def_arm_roll" value="0.0"/>  <!-- 0.4 -->
+	<property name="def_arm_pitch" value="0.785398"/> <!-- 0.7554 --> <!-- 0.785398 -->
+	<property name="def_arm_yaw" value="-2.1"/> <!-- -1.33899265359 --> <!-- -1.57 -->
 	<!-- pg70 mount positions | relative to arm_7_link -->
 	<property name="def_pg70_x" value="0.0"/>

File: cob_hardware_config/cob4-1/urdf/calibration_default.urdf.xacro (robot description, xacro)
@@ -45,36 +45,8 @@
 	<property name="def_sensorring_x" value="0.0"/>
 	<property name="def_sensorring_y" value="0.0"/>
-	<property name="def_sensorring_z" value="0.007"/>
+	<property name="def_sensorring_z" value="0.006"/>
 	<property name="def_sensorring_roll" value="0.0"/>
 	<property name="def_sensorring_pitch" value="0.0"/>
 	<property name="def_sensorring_yaw" value="0.0"/>
-	<!-- arm right mount positions | relative to torso_3_link -->
-	<property name="def_arm_right_x" value="0.0"/>
-	<property name="def_arm_right_y" value="-0.014"/>
-	<property name="def_arm_right_z" value="0.55"/>
-	<property name="def_arm_right_roll" value="1.57097"/>
-	<property name="def_arm_right_pitch" value="0"/>
-	<property name="def_arm_right_yaw" value="0.0"/>
-	<!-- arm left mount positions | relative to torso_3_link -->
-	<property name="def_arm_left_x" value="0.0"/>
-	<property name="def_arm_left_y" value="0.014"/>
-	<property name="def_arm_left_z" value="0.55"/>
-	<property name="def_arm_left_roll" value="1.57097"/>
-	<property name="def_arm_left_pitch" value="0"/>
-	<property name="def_arm_left_yaw" value="3.14159"/>
-	<!-- gripper right mount positions | relative to arm_right_7_link -->
-	<property name="def_gripper_right_x" value="0.0"/>
-	<property name="def_gripper_right_y" value="0.0"/>
-	<property name="def_gripper_right_z" value="0.0748"/>
-	<property name="def_gripper_right_roll" value="0.0"/>
-	<property name="def_gripper_right_pitch" value="0.0"/>
-	<property name="def_gripper_right_yaw" value="3.14159"/>
-	<!-- gripper left mount positions | relative to arm_left_7_link -->
-	<property name="def_gripper_left_x" value="0.0"/>
-	<property name="def_gripper_left_y" value="0.0"/>
-	<property name="def_gripper_left_z" value="0.0748"/>
-	<property name="def_gripper_left_roll" value="0.0"/>
-	<property name="def_gripper_left_pitch" value="0.0"/>
-	<property name="def_gripper_left_yaw" value="3.14159"/>
 	<!-- *********************************** -->
 	<!-- kinematic chain reference positions -->
@@ -102,3 +74,10 @@
 	<property name="def_torso_cam3d_down_pitch" value="0.0"/>
 	<property name="def_torso_cam3d_down_yaw" value="1.57079"/> <!--1.57079-->
+	<!-- cam3d | handeye calibration | relative to sensorring_link -->
+	<property name="def_sensorring_cam3d_x" value="0.096"/>
+	<property name="def_sensorring_cam3d_y" value="0.0"/>
+	<property name="def_sensorring_cam3d_z" value="0.0195"/>
+	<property name="def_sensorring_cam3d_roll" value="-1.5708"/>
+	<property name="def_sensorring_cam3d_pitch" value="0.0"/>
+	<property name="def_sensorring_cam3d_yaw" value="-1.5708"/>
 </robot>

File: cob_hardware_config/cob4-1/urdf/cob4-1.urdf.xacro (robot description, xacro)
@@ -11,16 +11,11 @@
   <xacro:include filename="$(find cob_description)/urdf/cob4_base/base.urdf.xacro" />
   <!-- torso -->
-  <xacro:include filename="$(find cob_description)/urdf/cob4_torso/torso_3dof.urdf.xacro" />
-  <xacro:include filename="$(find cob_description)/urdf/lookat/lookat.urdf.xacro" />
-  <!-- arm -->
-  <xacro:include filename="$(find schunk_description)/urdf/lwa4p_extended/lwa4p_extended.urdf.xacro" />
-  <!-- gripper -->
-  <xacro:include filename="$(find cob_description)/urdf/cob4_gripper/gripper.urdf.xacro" />
+  <xacro:include filename="$(find cob_description)/urdf/cob4_torso/torso_2dof.urdf.xacro" />
   <!-- head -->
   <xacro:include filename="$(find cob_description)/urdf/cob4_head/head.urdf.xacro" />
   <!-- sensorring -->
-  <xacro:include filename="$(find cob_description)/urdf/cob4_sensorring/sensorring.urdf.xacro" />
+  <xacro:include filename="$(find cob_description)/urdf/cob4_sensorring/sensorring_asus.urdf.xacro" />
   <!-- composition of the robot -->
-  <xacro:base name="base" use_old_joint_names="true"/>
+  <xacro:base name="base" use_old_joint_names="false"/>
   <gazebo>
     <plugin name="ros_control" filename="libhwi_switch_gazebo_ros_control.so">
@@ -56,46 +51,3 @@
     </plugin>
   </gazebo>
-  <xacro:schunk_lwa4p_extended name="arm_right" parent="torso_3_link" has_podest="false">
-    <origin xyz="${arm_right_x} ${arm_right_y} ${arm_right_z}" rpy="${arm_right_roll} ${arm_right_pitch} ${arm_right_yaw}" />
-  </xacro:schunk_lwa4p_extended>
-  <gazebo>
-    <plugin name="ros_control" filename="libhwi_switch_gazebo_ros_control.so">
-      <robotNamespace>arm_right</robotNamespace>
-      <filterJointsParam>joint_names</filterJointsParam>
-    </plugin>
-  </gazebo>
-  <xacro:schunk_lwa4p_extended name="arm_left" parent="torso_3_link" has_podest="false">
-    <origin xyz="${arm_left_x} ${arm_left_y} ${arm_left_z}" rpy="${arm_left_roll} ${arm_left_pitch} ${arm_left_yaw}" />
-  </xacro:schunk_lwa4p_extended>
-  <gazebo>
-    <plugin name="ros_control" filename="libhwi_switch_gazebo_ros_control.so">
-      <robotNamespace>arm_left</robotNamespace>
-      <filterJointsParam>joint_names</filterJointsParam>
-    </plugin>
-  </gazebo>
-  <xacro:gripper name="gripper_right" parent="arm_right_7_link">
-    <origin xyz="${gripper_right_x} ${gripper_right_y} ${gripper_right_z}" rpy="${gripper_right_roll} ${gripper_right_pitch} ${gripper_right_yaw}" />
-  </xacro:gripper>
-  <gazebo>
-    <plugin name="ros_control" filename="libhwi_switch_gazebo_ros_control.so">
-      <robotNamespace>gripper_right</robotNamespace>
-      <filterJointsParam>joint_names</filterJointsParam>
-    </plugin>
-  </gazebo>
-  <xacro:gripper name="gripper_left" parent="arm_left_7_link">
-    <origin xyz="${gripper_left_x} ${gripper_left_y} ${gripper_left_z}" rpy="${gripper_left_roll} ${gripper_left_pitch} ${gripper_left_yaw}" />
-  </xacro:gripper>
-  <gazebo>
-    <plugin name="ros_control" filename="libhwi_switch_gazebo_ros_control.so">
-      <robotNamespace>gripper_left</robotNamespace>
-      <filterJointsParam>joint_names</filterJointsParam>
-    </plugin>
-  </gazebo>
-  <!-- virtual component -->
-<!--
-  <xacro:lookat name="lookat" parent="torso_center_link" lower="0.0" upper="5.0">
-    <origin xyz="0 0 0" rpy="0 0 0" />
-    <axis xyz="1 0 0"/>
-  </xacro:lookat>
--->
 </robot>

File: cob_hardware_config/cob4-1/urdf/properties.urdf.xacro (robot description, xacro)
@@ -52,32 +52,4 @@
 	<property name="sensorring_pitch" value="${def_sensorring_pitch+offset_sensorring_pitch}"/>
 	<property name="sensorring_yaw" value="${def_sensorring_yaw+offset_sensorring_yaw}"/>
-	<!-- arm mount positions | relative to torso_3_link -->
-	<property name="arm_right_x" value="${def_arm_right_x+offset_arm_right_x}"/>
-	<property name="arm_right_y" value="${def_arm_right_y+offset_arm_right_y}"/>
-	<property name="arm_right_z" value="${def_arm_right_z+offset_arm_right_z}"/>
-	<property name="arm_right_roll" value="${def_arm_right_roll+offset_arm_right_roll}"/>
-	<property name="arm_right_pitch" value="${def_arm_right_pitch+offset_arm_right_pitch}"/>
-	<property name="arm_right_yaw" value="${def_arm_right_yaw+offset_arm_right_yaw}"/>
-	<!-- arm mount positions | relative to torso_3_link -->
-	<property name="arm_left_x" value="${def_arm_left_x+offset_arm_left_x}"/>
-	<property name="arm_left_y" value="${def_arm_left_y+offset_arm_left_y}"/>
-	<property name="arm_left_z" value="${def_arm_left_z+offset_arm_left_z}"/>
-	<property name="arm_left_roll" value="${def_arm_left_roll+offset_arm_left_roll}"/>
-	<property name="arm_left_pitch" value="${def_arm_left_pitch+offset_arm_left_pitch}"/>
-	<property name="arm_left_yaw" value="${def_arm_left_yaw+offset_arm_left_yaw}"/>
-	<!-- gripper right mount positions | relative to arm_right_7_link -->
-	<property name="gripper_right_x" value="${def_gripper_right_x+offset_gripper_right_x}"/>
-	<property name="gripper_right_y" value="${def_gripper_right_y+offset_gripper_right_y}"/>
-	<property name="gripper_right_z" value="${def_gripper_right_z+offset_gripper_right_z}"/>
-	<property name="gripper_right_roll" value="${def_gripper_right_roll+offset_gripper_right_roll}"/>
-	<property name="gripper_right_pitch" value="${def_gripper_right_pitch+offset_gripper_right_pitch}"/>
-	<property name="gripper_right_yaw" value="${def_gripper_right_yaw+offset_gripper_right_yaw}"/>
-	<!-- gripper left mount positions | relative to arm_left_7_link -->
-	<property name="gripper_left_x" value="${def_gripper_left_x+offset_gripper_left_x}"/>
-	<property name="gripper_left_y" value="${def_gripper_left_y+offset_gripper_left_y}"/>
-	<property name="gripper_left_z" value="${def_gripper_left_z+offset_gripper_left_z}"/>
-	<property name="gripper_left_roll" value="${def_gripper_left_roll+offset_gripper_left_roll}"/>
-	<property name="gripper_left_pitch" value="${def_gripper_left_pitch+offset_gripper_left_pitch}"/>
-	<property name="gripper_left_yaw" value="${def_gripper_left_yaw+offset_gripper_left_yaw}"/>
 	<!-- *********************************** -->
 	<!-- kinematic chain reference positions -->
@@ -105,3 +77,10 @@
 	<property name="torso_cam3d_down_pitch" value="${def_torso_cam3d_down_pitch+offset_torso_cam3d_down_pitch}"/>
 	<property name="torso_cam3d_down_yaw" value="${def_torso_cam3d_down_yaw+offset_torso_cam3d_down_yaw}"/>
+	<!-- cam3d | handeye calibration | relative to sensorring_link -->
+	<property name="sensorring_cam3d_x" value="${def_sensorring_cam3d_x+offset_sensorring_cam3d_x}"/>
+	<property name="sensorring_cam3d_y" value="${def_sensorring_cam3d_y+offset_sensorring_cam3d_y}"/>
+	<property name="sensorring_cam3d_z" value="${def_sensorring_cam3d_z+offset_sensorring_cam3d_z}"/>
+	<property name="sensorring_cam3d_roll" value="${def_sensorring_cam3d_roll+offset_sensorring_cam3d_roll}"/>
+	<property name="sensorring_cam3d_pitch" value="${def_sensorring_cam3d_pitch+offset_sensorring_cam3d_pitch}"/>
+	<property name="sensorring_cam3d_yaw" value="${def_sensorring_cam3d_yaw+offset_sensorring_cam3d_yaw}"/>
 </robot>

File: cob_hardware_config/cob4-2/urdf/calibration_default.urdf.xacro (robot description, xacro)
@@ -45,5 +45,5 @@
 	<property name="def_sensorring_x" value="0.0"/>
 	<property name="def_sensorring_y" value="0.0"/>
-	<property name="def_sensorring_z" value="0.007"/>
+	<property name="def_sensorring_z" value="0.006"/>
 	<property name="def_sensorring_roll" value="0.0"/>
 	<property name="def_sensorring_pitch" value="0.0"/>
@@ -102,3 +102,10 @@
 	<property name="def_torso_cam3d_down_pitch" value="0.0"/>
 	<property name="def_torso_cam3d_down_yaw" value="1.57079"/> <!--1.57079-->
+	<!-- cam3d | handeye calibration | relative to sensorring_link -->
+	<property name="def_sensorring_cam3d_x" value="0.096"/>
+	<property name="def_sensorring_cam3d_y" value="0.0"/>
+	<property name="def_sensorring_cam3d_z" value="0.0195"/>
+	<property name="def_sensorring_cam3d_roll" value="-1.5708"/>
+	<property name="def_sensorring_cam3d_pitch" value="0.0"/>
+	<property name="def_sensorring_cam3d_yaw" value="-1.5708"/>
 </robot>

File: cob_hardware_config/cob4-2/urdf/cob4-2.urdf.xacro (robot description, xacro)
@@ -12,5 +12,4 @@
   <!-- torso -->
   <xacro:include filename="$(find cob_description)/urdf/cob4_torso/torso_2dof.urdf.xacro" />
-  <xacro:include filename="$(find cob_description)/urdf/lookat/lookat.urdf.xacro" />
   <!-- arm -->
   <xacro:include filename="$(find schunk_description)/urdf/lwa4p_extended/lwa4p_extended.urdf.xacro" />
@@ -20,7 +19,7 @@
   <xacro:include filename="$(find cob_description)/urdf/cob4_head/head_static.urdf.xacro" />
   <!-- sensorring -->
-  <xacro:include filename="$(find cob_description)/urdf/cob4_sensorring/sensorring.urdf.xacro" />
+  <xacro:include filename="$(find cob_description)/urdf/cob4_sensorring/sensorring_asus.urdf.xacro" />
   <!-- composition of the robot -->
-  <xacro:base name="base" use_old_joint_names="true"/>
+  <xacro:base name="base" use_old_joint_names="false"/>
   <gazebo>
     <plugin name="ros_control" filename="libhwi_switch_gazebo_ros_control.so">
@@ -86,4 +85,3 @@
     </plugin>
   </gazebo>
-  <!-- virtual component -->
 </robot>

File: cob_hardware_config/cob4-2/urdf/properties.urdf.xacro (robot description, xacro)
@@ -105,3 +105,10 @@
 	<property name="torso_cam3d_down_pitch" value="${def_torso_cam3d_down_pitch+offset_torso_cam3d_down_pitch}"/>
 	<property name="torso_cam3d_down_yaw" value="${def_torso_cam3d_down_yaw+offset_torso_cam3d_down_yaw}"/>
+	<!-- cam3d | handeye calibration | relative to sensorring_link -->
+	<property name="sensorring_cam3d_x" value="${def_sensorring_cam3d_x+offset_sensorring_cam3d_x}"/>
+	<property name="sensorring_cam3d_y" value="${def_sensorring_cam3d_y+offset_sensorring_cam3d_y}"/>
+	<property name="sensorring_cam3d_z" value="${def_sensorring_cam3d_z+offset_sensorring_cam3d_z}"/>
+	<property name="sensorring_cam3d_roll" value="${def_sensorring_cam3d_roll+offset_sensorring_cam3d_roll}"/>
+	<property name="sensorring_cam3d_pitch" value="${def_sensorring_cam3d_pitch+offset_sensorring_cam3d_pitch}"/>
+	<property name="sensorring_cam3d_yaw" value="${def_sensorring_cam3d_yaw+offset_sensorring_cam3d_yaw}"/>
 </robot>

File: cob_hardware_config/raw3-1/urdf/raw3-1.urdf.xacro (robot description, xacro)
@@ -14,5 +14,4 @@
   <!-- head -->
   <xacro:include filename="$(find raw_description)/urdf/head/head.urdf.xacro" />
-  <xacro:include filename="$(find cob_description)/urdf/lookat/lookat.urdf.xacro" />
   <!-- ur_arm -->
   <xacro:include filename="$(find cob_description)/urdf/ur_arm/ur10_arm.urdf.xacro" />
@@ -42,8 +41,4 @@
     <origin xyz="${head_x} ${head_y} ${head_z}" rpy="${head_roll} ${head_pitch} ${head_yaw}" />
   </xacro:raw_head>
-  <!--xacro:cob_lookat name="lookat" parent="torso_2_link" lower="0.0" upper="5.0">
-    <origin xyz="${head_x} ${head_y} ${head_z}" rpy="${head_roll} ${head_pitch} ${head_yaw}" />
-    <axis xyz="1 0 0"/>
-  </xacro:cob_lookat-->
 <!--
   <xacro:ur10 name="arm" parent="base_link">

File: cob_hardware_config/raw3-3/urdf/raw3-3.urdf.xacro (robot description, xacro)
@@ -29,13 +29,7 @@
   <!-- prace macros -->
   <xacro:prace/>
-<!--
-  <xacro:lookat name="lookat" parent="head_cam_holder_link" lower="0.0" upper="8.0">
-    <origin xyz="${head_x} ${head_y} ${head_z}" rpy="${head_roll} ${head_pitch} ${head_yaw}" />
-    <axis xyz="1 0 0"/>
-  </xacro:lookat>
--->
   <!-- scan top mount -->
     <joint name="base_laser_top_joint" type="fixed" >
-      <origin xyz="0.28 0.0 0.885" rpy="0.0 0.0 ${M_PI}" />
+      <origin xyz="0.28 0.0 0.885" rpy="0.0 0.0 0.0" />
       <parent link="base_link" />
       <child link="base_laser_top_link" />
