Commit message: Imported upstream version '0.6.6' of 'upstream'

File: cob_hardware_config/cob4-1/urdf/calibration_default.urdf.xacro (robot description, xacro)
@@ -71,7 +71,7 @@
 	<property name="def_torso_cam3d_down_y" value="0.0"/>
 	<property name="def_torso_cam3d_down_z" value="0.14005"/>
-	<property name="def_torso_cam3d_down_roll" value="2.18166"/> <!--2.18166-->
-	<property name="def_torso_cam3d_down_pitch" value="0.0"/>
-	<property name="def_torso_cam3d_down_yaw" value="1.57079"/> <!--1.57079-->
+	<property name="def_torso_cam3d_down_roll" value="0.0"/>
+	<property name="def_torso_cam3d_down_pitch" value="0.54"/>
+	<property name="def_torso_cam3d_down_yaw" value="0.0"/>
 	<!-- cam3d | handeye calibration | relative to sensorring_link -->
 	<property name="def_sensorring_cam3d_x" value="0.096"/>

File: cob_hardware_config/cob4-1/urdf/cob4-1.urdf.xacro (robot description, xacro)
@@ -11,5 +11,5 @@
   <xacro:include filename="$(find cob_description)/urdf/cob4_base/base.urdf.xacro" />
   <!-- torso -->
-  <xacro:include filename="$(find cob_description)/urdf/cob4_torso/torso_2dof.urdf.xacro" />
+  <xacro:include filename="$(find cob_description)/urdf/cob4_torso/torso_2dof_realsense.urdf.xacro" />
   <!-- head -->
   <xacro:include filename="$(find cob_description)/urdf/cob4_head/head.urdf.xacro" />

File: cob_hardware_config/cob4-2/urdf/cob4-2.urdf.xacro (robot description, xacro)
@@ -17,5 +17,5 @@
   <xacro:include filename="$(find cob_description)/urdf/cob4_gripper/gripper.urdf.xacro" />
   <!-- head -->
-  <xacro:include filename="$(find cob_description)/urdf/cob4_head/head_static.urdf.xacro" />
+  <xacro:include filename="$(find cob_description)/urdf/cob4_head/head.urdf.xacro" />
   <!-- sensorring -->
   <xacro:include filename="$(find cob_description)/urdf/cob4_sensorring/sensorring_asus.urdf.xacro" />
@@ -40,4 +40,10 @@
     <origin xyz="${head_x} ${head_y} ${head_z}" rpy="${head_roll} ${head_pitch} ${head_yaw}" />
   </xacro:head>
+  <gazebo>
+    <plugin name="ros_control" filename="libhwi_switch_gazebo_ros_control.so">
+      <robotNamespace>head</robotNamespace>
+      <filterJointsParam>joint_names</filterJointsParam>
+    </plugin>
+  </gazebo>
   <xacro:sensorring name="sensorring" parent="head_3_link">
     <origin xyz="${sensorring_x} ${sensorring_y} ${sensorring_z}" rpy="${sensorring_roll} ${sensorring_pitch} ${sensorring_yaw}" />

File: cob_hardware_config/raw3-6/urdf/calibration_default.urdf.xacro (robot description, xacro)
@@ -28,3 +28,10 @@
 	<property name="def_tower_pitch" value="0.0"/>
 	<property name="def_tower_yaw" value="0.0"/>
+	<!--arm mount positions | relative to base_link-->
+	<property name="def_arm_x" value="0.330"/>
+	<property name="def_arm_y" value="0.0"/>
+	<property name="def_arm_z" value="0.482"/>
+	<property name="def_arm_roll" value="0.0"/>
+	<property name="def_arm_pitch" value="0.0"/>
+	<property name="def_arm_yaw" value="${-M_PI/2}"/>
 </robot>

File: cob_hardware_config/raw3-6/urdf/properties.urdf.xacro (robot description, xacro)
@@ -30,3 +30,10 @@
 	<property name="tower_pitch" value="${def_tower_pitch+offset_tower_pitch}"/>
 	<property name="tower_yaw" value="${def_tower_yaw+offset_tower_yaw}"/>
+	<!-- arm mount positions | relative to base_link -->
+	<property name="arm_x" value="${def_arm_x+offset_arm_x}"/>
+	<property name="arm_y" value="${def_arm_y+offset_arm_y}"/>
+	<property name="arm_z" value="${def_arm_z+offset_arm_z}"/>
+	<property name="arm_roll" value="${def_arm_roll+offset_arm_roll}"/>
+	<property name="arm_pitch" value="${def_arm_pitch+offset_arm_pitch}"/>
+	<property name="arm_yaw" value="${def_arm_yaw+offset_arm_yaw}"/>
 </robot>

File: cob_hardware_config/raw3-6/urdf/raw3-6.urdf.xacro (robot description, xacro)
@@ -10,4 +10,6 @@
   <!-- raw tower -->
   <xacro:include filename="$(find raw_description)/urdf/tower_symetric/tower.urdf.xacro" />
+  <!-- ur10 -->
+  <xacro:include filename="$(find cob_description)/urdf/ur_arm/ur10_arm.urdf.xacro" />
   <!-- composition of the robot -->
   <xacro:raw_base name="base"/>
@@ -21,3 +23,12 @@
       <origin xyz="${tower_x} ${tower_y} ${tower_z}" rpy="${tower_roll} ${tower_pitch} ${tower_yaw}" />
   </xacro:tower_symetric>
+  <xacro:ur10 name="arm" parent="base_link">
+    <origin xyz="${arm_x} ${arm_y} ${arm_z}" rpy="${arm_roll} ${arm_pitch} ${arm_yaw}" />
+  </xacro:ur10>
+  <gazebo>
+    <plugin name="ros_control" filename="libhwi_switch_gazebo_ros_control.so">
+      <robotNamespace>arm</robotNamespace>
+      <filterJointsParam>joint_names</filterJointsParam>
+    </plugin>
+  </gazebo>
   </robot>
